Commit message: convert URDFs without Collada files to use relative path instead of "package://" in model references.

File: urdf_files/matlab/abb_irb120_support/urdf/abbIrb120.urdf (robot description, URDF)
Before this commit: robot abb_irb120_3_58, 9 links, 8 joints
Links:
- link base_link: geometry collision mesh filename=../../abb_irb120_support/meshes/irb120_3_58/collision/base_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; visual mesh filename=../../abb_irb120_support/meshes/irb120_3_58/visual/base_lin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
- link link_1: geometry collision mesh filename=../../abb_irb120_support/meshes/irb120_3_58/collision/link_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; visual mesh filename=../../abb_irb120_support/meshes/irb120_3_58/visual/link_1.s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
- link link_2: geometry collision mesh filename=../../abb_irb120_support/meshes/irb120_3_58/collision/link_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; visual mesh filename=../../abb_irb120_support/meshes/irb120_3_58/visual/link_2.s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
- link link_3: geometry collision mesh filename=../../abb_irb120_support/meshes/irb120_3_58/collision/link_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; visual mesh filename=../../abb_irb120_support/meshes/irb120_3_58/visual/link_3.s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
- link link_4: geometry collision mesh filename=../../abb_irb120_support/meshes/irb120_3_58/collision/link_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; visual mesh filename=../../abb_irb120_support/meshes/irb120_3_58/visual/link_4.s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
- link link_5: geometry collision mesh filename=../../abb_irb120_support/meshes/irb120_3_58/collision/link_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; visual mesh filename=../../abb_irb120_support/meshes/irb120_3_58/visual/link_5.s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
- link link_6: geometry collision mesh filename=../../abb_irb120_support/meshes/irb120_3_58/collision/link_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; visual mesh filename=../../abb_irb120_support/meshes/irb120_3_58/visual/link_6.s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

File: urdf_files/matlab/abb_irb1600_support/urdf/abbIrb1600.urdf (robot description, URDF)
Before this commit: robot abb_irb1600_6_12, 8 links, 7 joints
Links:
- link base_link: geometry collision mesh filename=../../abb_irb1600_support/meshes/irb1600/collision/base_lin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; visual mesh filename=../../abb_irb1600_support/meshes/irb1600/visual/base_link.s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
- link link_1: geometry collision mesh filename=../../abb_irb1600_support/meshes/irb1600/collision/link_1.s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; visual mesh filename=../../abb_irb1600_support/meshes/irb1600/visual/link_1.stl
- link link_2: geometry collision mesh filename=../../abb_irb1600_support/meshes/irb1600_6_12/collision/lin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; visual mesh filename=../../abb_irb1600_support/meshes/irb1600_6_12/visual/link_2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
- link link_3: geometry collision mesh filename=../../abb_irb1600_support/meshes/irb1600/collision/link_3.s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; visual mesh filename=../../abb_irb1600_support/meshes/irb1600/visual/link_3.stl
- link link_4: geometry collision mesh filename=../../abb_irb1600_support/meshes/irb1600/collision/link_4.s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; visual mesh filename=../../abb_irb1600_support/meshes/irb1600/visual/link_4.stl
- link link_5: geometry collision mesh filename=../../abb_irb1600_support/meshes/irb1600/collision/link_5.s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; visual mesh filename=../../abb_irb1600_support/meshes/irb1600/visual/link_5.stl
- link link_6: geometry collision mesh filename=../../abb_irb1600_support/meshes/irb1600/collision/link_6.s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; visual mesh filename=../../abb_irb1600_support/meshes/irb1600/visual/link_6.stl

File: urdf_files/matlab/fanuc_lrmate200ib_support/urdf/fanucLRMate200ib.urdf (robot description, URDF)
Before this commit: robot fanuc_lrmate200ib, 10 links, 9 joints
Links:
- link base_link: geometry collision mesh filename=../../fanuc_lrmate200ib_support/meshes/lrmate200ib/collisio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; visual mesh filename=../../fanuc_lrmate200ib_support/meshes/lrmate200ib/visual/b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
- link link_1: geometry collision mesh filename=../../fanuc_lrmate200ib_support/meshes/lrmate200ib/collisio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; visual mesh filename=../../fanuc_lrmate200ib_support/meshes/lrmate200ib/visual/l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
- link link_2: geometry collision mesh filename=../../fanuc_lrmate200ib_support/meshes/lrmate200ib/collisio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; visual mesh filename=../../fanuc_lrmate200ib_support/meshes/lrmate200ib/visual/l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
- link link_3: geometry collision mesh filename=../../fanuc_lrmate200ib_support/meshes/lrmate200ib/collisio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; visual mesh filename=../../fanuc_lrmate200ib_support/meshes/lrmate200ib/visual/l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
- link link_4: geometry collision mesh filename=../../fanuc_lrmate200ib_support/meshes/lrmate200ib/collisio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; visual mesh filename=../../fanuc_lrmate200ib_support/meshes/lrmate200ib/visual/l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
- link link_5: geometry collision mesh filename=../../fanuc_lrmate200ib_support/meshes/lrmate200ib/collisio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; visual mesh filename=../../fanuc_lrmate200ib_support/meshes/lrmate200ib/visual/l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
- link link_6: geometry collision mesh filename=../../fanuc_lrmate200ib_support/meshes/lrmate200ib/collisio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; visual mesh filename=../../fanuc_lrmate200ib_support/meshes/lrmate200ib/visual/l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

File: urdf_files/matlab/fanuc_m16ib_support/urdf/fanucM16ib.urdf (robot description, URDF)
Before this commit: robot fanuc_m16ib20, 8 links, 7 joints
Links:
- link base_link: geometry collision mesh filename=../../fanuc_m16ib_support/meshes/m16ib20/collision/base_lin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; visual mesh filename=../../fanuc_m16ib_support/meshes/m16ib20/visual/base_link.s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
- link link_1: geometry collision mesh filename=../../fanuc_m16ib_support/meshes/m16ib20/collision/link_1.s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; visual mesh filename=../../fanuc_m16ib_support/meshes/m16ib20/visual/link_1.stl
- link link_2: geometry collision mesh filename=../../fanuc_m16ib_support/meshes/m16ib20/collision/link_2.s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; visual mesh filename=../../fanuc_m16ib_support/meshes/m16ib20/visual/link_2.stl
- link link_3: geometry collision mesh filename=../../fanuc_m16ib_support/meshes/m16ib20/collision/link_3.s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; visual mesh filename=../../fanuc_m16ib_support/meshes/m16ib20/visual/link_3.stl
- link link_4: geometry collision mesh filename=../../fanuc_m16ib_support/meshes/m16ib20/collision/link_4.s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; visual mesh filename=../../fanuc_m16ib_support/meshes/m16ib20/visual/link_4.stl
- link link_5: geometry collision mesh filename=../../fanuc_m16ib_support/meshes/m16ib20/collision/link_5.s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; visual mesh filename=../../fanuc_m16ib_support/meshes/m16ib20/visual/link_5.stl
- link link_6: geometry collision mesh filename=../../fanuc_m16ib_support/meshes/m16ib20/collision/link_6.s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; visual mesh filename=../../fanuc_m16ib_support/meshes/m16ib20/visual/link_6.stl

File: urdf_files/matlab/iiwa_description/urdf/kukaIiwa14.urdf (robot description, URDF)
Before this commit: robot iiwa14, 11 links, 10 joints
Links:
- link iiwa_link_0: geometry collision mesh filename=../../iiwa_description/meshes/iiwa14/collision/link_0.stl; visual mesh filename=../../iiwa_description/meshes/iiwa14/visual/link_0.stl
- link iiwa_link_1: geometry collision mesh filename=../../iiwa_description/meshes/iiwa14/collision/link_1.stl; visual mesh filename=../../iiwa_description/meshes/iiwa14/visual/link_1.stl
- link iiwa_link_2: geometry collision mesh filename=../../iiwa_description/meshes/iiwa14/collision/link_2.stl; visual mesh filename=../../iiwa_description/meshes/iiwa14/visual/link_2.stl
- link iiwa_link_3: geometry collision mesh filename=../../iiwa_description/meshes/iiwa14/collision/link_3.stl; visual mesh filename=../../iiwa_description/meshes/iiwa14/visual/link_3.stl
- link iiwa_link_4: geometry collision mesh filename=../../iiwa_description/meshes/iiwa14/collision/link_4.stl; visual mesh filename=../../iiwa_description/meshes/iiwa14/visual/link_4.stl
- link iiwa_link_5: geometry collision mesh filename=../../iiwa_description/meshes/iiwa14/collision/link_5.stl; visual mesh filename=../../iiwa_description/meshes/iiwa14/visual/link_5.stl
- link iiwa_link_6: geometry collision mesh filename=../../iiwa_description/meshes/iiwa14/collision/link_6.stl; visual mesh filename=../../iiwa_description/meshes/iiwa14/visual/link_6.stl
- link iiwa_link_7: geometry collision mesh filename=../../iiwa_description/meshes/iiwa14/collision/link_7.stl; visual mesh filename=../../iiwa_description/meshes/iiwa14/visual/link_7.stl

File: urdf_files/matlab/iiwa_description/urdf/kukaIiwa7.urdf (robot description, URDF)
Before this commit: robot iiwa7, 11 links, 10 joints
Links:
- link iiwa_link_0: geometry collision mesh filename=../../iiwa_description/meshes/iiwa7/collision/link_0.stl; visual mesh filename=../../iiwa_description/meshes/iiwa7/visual/link_0.stl
- link iiwa_link_1: geometry collision mesh filename=../../iiwa_description/meshes/iiwa7/collision/link_1.stl; visual mesh filename=../../iiwa_description/meshes/iiwa7/visual/link_1.stl
- link iiwa_link_2: geometry collision mesh filename=../../iiwa_description/meshes/iiwa7/collision/link_2.stl; visual mesh filename=../../iiwa_description/meshes/iiwa7/visual/link_2.stl
- link iiwa_link_3: geometry collision mesh filename=../../iiwa_description/meshes/iiwa7/collision/link_3.stl; visual mesh filename=../../iiwa_description/meshes/iiwa7/visual/link_3.stl
- link iiwa_link_4: geometry collision mesh filename=../../iiwa_description/meshes/iiwa7/collision/link_4.stl; visual mesh filename=../../iiwa_description/meshes/iiwa7/visual/link_4.stl
- link iiwa_link_5: geometry collision mesh filename=../../iiwa_description/meshes/iiwa7/collision/link_5.stl; visual mesh filename=../../iiwa_description/meshes/iiwa7/visual/link_5.stl
- link iiwa_link_6: geometry collision mesh filename=../../iiwa_description/meshes/iiwa7/collision/link_6.stl; visual mesh filename=../../iiwa_description/meshes/iiwa7/visual/link_6.stl
- link iiwa_link_7: geometry collision mesh filename=../../iiwa_description/meshes/iiwa7/collision/link_7.stl; visual mesh filename=../../iiwa_description/meshes/iiwa7/visual/link_7.stl

File: urdf_files/matlab/motoman_mh5_support/urdf/yaskawaMotomanMH5.urdf (robot description, URDF)
Before this commit: robot motoman_mh5, 7 links, 6 joints
Links:
- link base_link: geometry collision mesh filename=../../motoman_mh5_support/meshes/mh5/collision/MH5_BASE_AXI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; visual mesh filename=../../motoman_mh5_support/meshes/mh5/visual/MH5_BASE_AXIS.s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
- link link_b: geometry collision mesh filename=../../motoman_mh5_support/meshes/mh5/collision/MH5_B_AXIS.s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; visual mesh filename=../../motoman_mh5_support/meshes/mh5/visual/MH5_B_AXIS.stl
- link link_l: geometry collision mesh filename=../../motoman_mh5_support/meshes/mh5/collision/MH5_L_AXIS.s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; visual mesh filename=../../motoman_mh5_support/meshes/mh5/visual/MH5_L_AXIS.stl
- link link_r: geometry collision mesh filename=../../motoman_mh5_support/meshes/mh5/collision/MH5_R_AXIS.s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; visual mesh filename=../../motoman_mh5_support/meshes/mh5/visual/MH5_R_AXIS.stl
- link link_s: geometry collision mesh filename=../../motoman_mh5_support/meshes/mh5/collision/MH5_S_AXIS.s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; visual mesh filename=../../motoman_mh5_support/meshes/mh5/visual/MH5_S_AXIS.stl
- link link_t: geometry collision mesh filename=../../motoman_mh5_support/meshes/mh5/collision/MH5_T_AXIS.s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; visual mesh filename=../../motoman_mh5_support/meshes/mh5/visual/MH5_T_AXIS.stl
- link link_u: geometry collision mesh filename=../../motoman_mh5_support/meshes/mh5/collision/MH5_U_AXIS.s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; visual mesh filename=../../motoman_mh5_support/meshes/mh5/visual/MH5_U_AXIS.stl

File: urdf_files/robotics-toolbox/abb_irb140/urdf/irb140.urdf (robot description, URDF)
Before this commit: robot abb_irb140, 9 links, 8 joints
Links:
- link base_link: geometry collision mesh filename=../../abb_irb140/meshes/irb140/collision/base_link.stl; visual mesh filename=../../abb_irb140/meshes/irb140/visual/base_link.stl
- link link_1: geometry collision mesh filename=../../abb_irb140/meshes/irb140/collision/link_1.stl; visual mesh filename=../../abb_irb140/meshes/irb140/visual/link_1.stl
- link link_2: geometry collision mesh filename=../../abb_irb140/meshes/irb140/collision/link_2.stl; visual mesh filename=../../abb_irb140/meshes/irb140/visual/link_2.stl
- link link_3: geometry collision mesh filename=../../abb_irb140/meshes/irb140/collision/link_3.stl; visual mesh filename=../../abb_irb140/meshes/irb140/visual/link_3.stl
- link link_4: geometry collision mesh filename=../../abb_irb140/meshes/irb140/collision/link_4.stl; visual mesh filename=../../abb_irb140/meshes/irb140/visual/link_4.stl
- link link_5: geometry collision mesh filename=../../abb_irb140/meshes/irb140/collision/link_5.stl; visual mesh filename=../../abb_irb140/meshes/irb140/visual/link_5.stl
- link link_6: geometry collision mesh filename=../../abb_irb140/meshes/irb140/collision/link_6.stl; visual mesh filename=../../abb_irb140/meshes/irb140/visual/link_6.stl

File: urdf_files/ros-industrial/abb/abb_irb5400_support/urdf/irb5400.urdf (robot description, URDF)
Before this commit: robot abb_irb5400, 10 links, 9 joints
Links:
- link base_link: geometry collision mesh filename=../meshes/collision/base_link.stl; visual mesh filename=../meshes/visual/base_link.dae
- link link_1: geometry collision mesh filename=../meshes/collision/link_1.stl; visual mesh filename=../meshes/visual/link_1.dae
- link link_2: geometry collision mesh filename=../meshes/collision/link_2.stl; visual mesh filename=../meshes/visual/link_2.dae
- link link_3: geometry collision mesh filename=../meshes/collision/link_3.stl; visual mesh filename=../meshes/visual/link_3.dae
- link link_4: geometry collision mesh filename=../meshes/collision/link_4.stl; visual mesh filename=../meshes/visual/link_4.dae
- link link_5: geometry collision mesh filename=../meshes/collision/link_5.stl; visual mesh filename=../meshes/visual/link_5.dae
- link link_5b: geometry collision mesh filename=../meshes/collision/link_5b.stl; visual mesh filename=../meshes/visual/link_5b.dae
- link link_6: geometry collision mesh filename=../meshes/collision/link_6.stl; visual mesh filename=../meshes/visual/link_6.dae
