Commit message: turtlebot3

File: urdf_files/oems/xacro_generated/turtlebot3_robotis/turtlebot3_description/urdf/turtlebot3_burger.urdf (robot description, URDF)
Before this commit: robot turtlebot3_burger, 7 links, 6 joints
Links:
- link base_link: geometry collision box size=0.140 0.140 0.143; visual mesh filename=../../turtlebot3_description/meshes/bases/burger_base.stl scale=0.001 0.001 0.001
- link base_scan: geometry collision cylinder length=0.0315 radius=0.055; visual mesh filename=../../turtlebot3_description/meshes/sensors/lds.stl scale=0.001 0.001 0.001
- link wheel_left_link: geometry collision cylinder length=0.018 radius=0.033; visual mesh filename=../../turtlebot3_description/meshes/wheels/left_tire.stl scale=0.001 0.001 0.001
- link wheel_right_link: geometry collision cylinder length=0.018 radius=0.033; visual mesh filename=../../turtlebot3_description/meshes/wheels/right_tire.stl scale=0.001 0.001 0.001
